File: Famicom composite.kicad_pcb (KiCad board)
At the start: 2 copper layers, 14.2 x 19.9 mm, 11 parts, among them J1 PPU_Pin21, J2 Conn_01x02, J3 Audio_In, J4 Conn_01x04_Female, U1 THS7314

Commit message: Update to KiCad 7
Other:
- net class Default removed

Commit message: Release v0.6
Other:
- rule pad_to_mask_clearance: 0.051 -> 0
Changed lines of the file:
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@@
   )
   (setup
-    (pad_to_mask_clearance 0.051)
-    (solder_mask_min_width 0.25)
+    (pad_to_mask_clearance 0)
     (pcbplotparams
       (layerselection 0x00010fc_ffffffff)
